Commit message: modified diff_drive

File: diff_drive/urdf/ddrive.urdf.xacro (robot description, xacro)
@@ -23,7 +23,7 @@
       <origin xyz="0.0 0 0.0" rpy=" 0 0 0"/>
       <inertia
-          ixx="0.1" ixy="0" ixz="0"
-          iyy="0.1" iyz="0"
-          izz="0.1"
+          ixx="0.1305" ixy="0" ixz="0"
+          iyy="0.3305" iyz="0"
+          izz="0.425"
       />
     </inertial>
@@ -67,10 +67,10 @@
  <link name='left_wheel'>
     <inertial>
-      <mass value="2.0"/>
+      <mass value="5.0"/>
       <origin xyz="0.0 0 0.0" rpy=" 0 1.5707 1.5707"/>
       <inertia
-          ixx="0.1" ixy="0" ixz="0"
-          iyy="0.1" iyz="0"
-          izz="0.1"
+          ixx="0.027" ixy="0" ixz="0"
+          iyy="0.027" iyz="0"
+          izz="0.048"
       />
     </inertial>
@@ -90,10 +90,10 @@
 <link name='right_wheel'>
     <inertial>
-      <mass value="2.0"/>
+      <mass value="5.0"/>
       <origin xyz="0.0 0 0.0" rpy=" 0 1.5707 1.5707"/>
       <inertia
-          ixx="0.1" ixy="0" ixz="0"
-          iyy="0.1" iyz="0"
-          izz="0.1"
+          ixx="0.027" ixy="0" ixz="0"
+          iyy="0.027" iyz="0"
+          izz="0.048"
       />
     </inertial>

Commit message: added README

File: diff_drive/urdf/ddrive.urdf.xacro (robot description, xacro)
@@ -18,12 +18,12 @@
   </joint>
   <link name='chassis'>
-    <pose>0 0 0 0 0 0</pose>
+    <pose>0 0 0.0 0 0 0</pose>
     <inertial>
-      <mass value="15.0"/>
+      <mass value="5.0"/>
       <origin xyz="0.0 0 0.0" rpy=" 0 0 0"/>
       <inertia
-          ixx="0.1305" ixy="0" ixz="0"
-          iyy="0.3305" iyz="0"
-          izz="0.425"
+          ixx="0.1" ixy="0" ixz="0"
+          iyy="0.1" iyz="0"
+          izz="0.1"
       />
     </inertial>
@@ -40,6 +40,17 @@
       </geometry>
     </visual>
+  </link>
+<link name='bottom_caster'>
+    <inertial>
+      <mass value="0"/>
+      <origin xyz="0 0 0" rpy=" 0 0 0"/>
+      <inertia
+          ixx="0.0" ixy="0" ixz="0"
+          iyy="0.0" iyz="0"
+          izz="0.0"
+      />
+    </inertial>
     <collision name='bottom_caster_collision'>
-      <origin xyz="-0.20 0 -0.05" rpy=" 0 0 0"/>
+      <origin xyz="0 0 0" rpy=" 0 0 0"/>
       <geometry>
         <sphere radius="${R2}"/>
@@ -47,11 +58,22 @@
     </collision>
     <visual name='bottom_caster_visual'>
-      <origin xyz="-0.20 0 -0.05" rpy=" 0 0 0"/>
+      <origin xyz="0 0 0" rpy=" 0 0 0"/>
       <geometry>
         <sphere radius="${R2}"/>
       </geometry>
     </visual>
+</link>
+<link name='top_caster'>
+    <inertial>
+      <mass value="0.0"/>
+      <origin xyz="0 0 0" rpy=" 0 0 0"/>
+      <inertia
+          ixx="0.0" ixy="0" ixz="0"
+          iyy="0.0" iyz="0"
+          izz="0.0"
+      />
+    </inertial>
     <collision name='top_caster_collision'>
-      <origin xyz="-0.20 0 0.05" rpy=" 0 0 0"/>
+      <origin xyz="0 0 0" rpy=" 0 0 0"/>
       <geometry>
         <sphere radius="${R2}"/>
@@ -59,18 +81,18 @@
     </collision>
     <visual name='top_caster_visual'>
-      <origin xyz="-0.20 0 0.05" rpy=" 0 0 0"/>
+      <origin xyz="0 0 0" rpy=" 0 0 0"/>
       <geometry>
         <sphere radius="${R2}"/>
       </geometry>
     </visual>
-  </link>
+</link>
  <link name='left_wheel'>
     <inertial>
-      <mass value="5.0"/>
+      <mass value="8"/>
       <origin xyz="0.0 0 0.0" rpy=" 0 1.5707 1.5707"/>
       <inertia
-          ixx="0.027" ixy="0" ixz="0"
-          iyy="0.027" iyz="0"
-          izz="0.048"
+          ixx="0.1" ixy="0" ixz="0"
+          iyy="0.1" iyz="0"
+          izz="0.1"
       />
     </inertial>
@@ -78,5 +100,5 @@
       <origin xyz="0 0 0.0" rpy=" 0 1.5707 1.5707"/>
       <geometry>
-        <cylinder radius="${r}" length="${l}"/>
+        <cylinder radius = "${r}" length = "${l}" />
       </geometry>
     </collision>
@@ -90,10 +112,10 @@
 <link name='right_wheel'>
     <inertial>
-      <mass value="5.0"/>
+      <mass value="8.0"/>
       <origin xyz="0.0 0 0.0" rpy=" 0 1.5707 1.5707"/>
       <inertia
-          ixx="0.027" ixy="0" ixz="0"
-          iyy="0.027" iyz="0"
-          izz="0.048"
+          ixx="0.1" ixy="0" ixz="0"
+          iyy="0.1" iyz="0"
+          izz="0.1"
       />
     </inertial>
@@ -110,28 +132,28 @@
       </geometry>
     </visual>
-</link>
+</link> -->
   <joint type="continuous" name="left_wheel_hinge">
-    <origin xyz="0.14 0.18 0" rpy="0 0 0"/>
+    <origin xyz="-0.14 0.18 0" rpy="0 0 0"/>
     <child link="left_wheel"/>
     <parent link="chassis"/>
     <axis xyz="0 1 0" rpy="0 0 0"/>
-    <mu1>1</mu1>
-    <mu2>1</mu2>
-    <kp>500000.0</kp>
-    <kd>10.0</kd>
-    <minDepth>0.001</minDepth>
-    <maxVel>0.1</maxVel>
   </joint>
-  <joint type="continuous" name="right_wheel_hinge">
-    <origin xyz="0.14 -0.18 0" rpy="0 0 0"/>
+   <joint type="continuous" name="right_wheel_hinge">
+    <origin xyz="-0.14 -0.18 0" rpy="0 0 0"/>
     <child link="right_wheel"/>
     <parent link="chassis"/>
     <axis xyz="0 1 0" rpy="0 0 0"/>
-    <mu1>1</mu1>
-    <mu2>1</mu2>
-    <kp>500000.0</kp>
-    <kd>10.0</kd>
-    <minDepth>0.001</minDepth>
-    <maxVel>0.1</maxVel>
+  </joint>
+  <joint type="fixed" name="bottom_caster_joint">
+    <origin xyz="0.20 0 -0.05" rpy="0 0 0"/>
+    <child link="bottom_caster"/>
+    <parent link="chassis"/>
+    <axis xyz="1 0 0" rpy="0 0 0"/>
+  </joint>
+  <joint type="fixed" name="top_caster_joint">
+    <origin xyz="0.20 0 0.05" rpy="0 0 0"/>
+    <child link="top_caster"/>
+    <parent link="chassis"/>
+    <axis xyz="1 0 0" rpy="0 0 0"/>
   </joint>
 </robot>

Commit message: modified readme

File: diff_drive/urdf/ddrive.urdf.xacro (robot description, xacro)
@@ -3,4 +3,5 @@
 <xacro:property name="yaml_file" value="$(find diff_drive)/config/ddrive.yaml" />
 <xacro:property name="robot_param" value="${load_yaml(yaml_file)}"/>
+<xacro:property name="M" value="${robot_param['M']}" />
 <xacro:property name="L" value="${robot_param['L']}" />
 <xacro:property name="W" value="${robot_param['W']}" />
@@ -10,4 +11,5 @@
 <xacro:property name="r" value="${robot_param['r']}" />
 <xacro:property name="l" value="${robot_param['l']}" />
+<xacro:property name="m" value="${robot_param['m']}" />
 <xacro:include filename="$(find diff_drive)/urdf/ddrive.gazebo" />
   <link name="base_link"></link>
@@ -20,5 +22,5 @@
     <pose>0 0 0.0 0 0 0</pose>
     <inertial>
-      <mass value="5.0"/>
+      <mass value="${M}"/>
       <origin xyz="0.0 0 0.0" rpy=" 0 0 0"/>
       <inertia
@@ -89,5 +91,5 @@
  <link name='left_wheel'>
     <inertial>
-      <mass value="8"/>
+      <mass value="${m}"/>
       <origin xyz="0.0 0 0.0" rpy=" 0 1.5707 1.5707"/>
       <inertia
@@ -112,5 +114,5 @@
 <link name='right_wheel'>
     <inertial>
-      <mass value="8.0"/>
+      <mass value="${m}"/>
       <origin xyz="0.0 0 0.0" rpy=" 0 1.5707 1.5707"/>
       <inertia
